File: current_sensor.kicad_sch (KiCad schematic)
At the start: 1 part

Commit message: updated the schematic diagram
Connections:
- net LOAD is gone; now on net OUT: U1. (GND)
- net SUPPLY is gone; now on net OUT: U1. (GND)
- net GPIO 14 renamed OUT
- new net CURRENT OUTPUT: U1. (GND)
- new net IN: U1. (GND)
Changed lines of the file:
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@@
 	(wire
 		(pts
-			(xy 116.84 85.09) (xy 133.35 85.09)
+			(xy 158.75 83.82) (xy 165.1 83.82)
 		)
 		(stroke
@@
 	(wire
 		(pts
-			(xy 158.75 83.82) (xy 162.56 83.82)
+			(xy 165.1 83.82) (xy 165.1 77.47)
 		)
 		(stroke
@@
 		)
 	)
-	(label "LOAD"
-		(at 118.11 88.9 0)
+	(wire
+		(pts
+			(xy 118.11 85.09) (xy 133.35 85.09)
+		)
+		(stroke
+			(width 0)
+			(type default)
+		)
+	)
+	(label "IN"
+		(at 119.38 85.09 0)
 		(effects
 			(font
@@
 		)
 	)
-	(label "GPIO 14"
+	(label "CURRENT OUTPUT"
 		(at 171.45 86.36 0)
 		(effects
@@
 		)
 	)
-	(label "SUPPLY"
-		(at 118.11 85.09 0)
-		(effects
-			(font
-				(size 1.27 1.27)
-			)
-			(justify left bottom)
-		)
-	)
-	(label "5V"
-		(at 160.02 83.82 0)
+	(label "OUT"
+		(at 118.11 88.9 0)
 		(effects
 			(font
@@
 					(unit 1)
 				)
+			)
+		)
+	)
+	(symbol
+		(lib_id "power:VCC")
+		(at 165.1 77.47 0)
+		(unit 1)
+		(exclude_from_sim no)
+		(in_bom yes)
+		(on_board yes)
+		(dnp no)
+		(fields_autoplaced yes)
+		(property "Reference" "#PWR02"
+			(at 165.1 81.28 0)
+			(effects
+				(font
+					(size 1.27 1.27)
+				)
+				(hide yes)
+			)
+		)
+		(property "Value" "5V"
+			(at 165.1 72.39 0)
+			(effects
+				(font
+					(size 1.27 1.27)
+				)
+			)
+		)
+		(property "Footprint" ""
+			(at 165.1 77.47 0)
+			(effects
+				(font
+					(size 1.27 1.27)
+				)
+				(hide yes)
+			)
+		)
+		(property "Datasheet" ""
+			(at 165.1 77.47 0)
+			(effects
+				(font
+					(size 1.27 1.27)
+				)
+				(hide yes)
+			)
+		)
+		(property "Description" "Power symbol creates a global label with name \"VCC\""
+			(at 165.1 77.47 0)
+			(effects
+				(font
+					(size 1.27 1.27)
+				)
+				(hide yes)
+			)
+		)
+		(pin "1"
+		)
+		(instances
+			(project ""
+				(path "/7255cc6b-4b58-46c5-a322-1ec6c681096b/baaf7afa-144d-4451-a089-126e571b21ae"
+					(reference "#PWR02")
+					(unit 1)
+				)
