File: current_sensor_schematic.kicad_sch (KiCad schematic)
At the start: 1 part

Commit message: schematic_merged
Parts:
- added U10: ZC261500, custom:MODULE_ZC261500, symbol ADS1115_module:ZC261500
- added U11, U13, U7: ~, symbol ASC712_current_sensor:ASC712_Current_sensor
Connections:
- net CURRENT OUTPUT is gone; now on net OUT: U5. (GND)
- net 5V: now also U10.10 (VDD), U11. (GND), U13. (GND), U7. (GND)
- net GND: now also U10.9 (GND), U11. (GND), U13. (GND), U7. (GND)
- net IN: now also U11. (GND), U13. (GND), U7. (GND)
- net OUT: now also U11. (GND), U13. (GND), U7. (GND)
- no-connect marks 0 -> 2
Other:
- note added: "the SDA is connected to GPio 21(D21) and the SCL is connected to GPI22 VDD go to 5v supply GND connected to common GND The ADC pin is then connected to the vout of the ACS712 (current sensor) the IP- is connected to possitve of the pump the IP+ is connected to possitve of the power supply"
- moved on the sheet: U5
