File: relay_schematic.kicad_sch (KiCad schematic)
At the start: 5 parts

Commit message: schematic_merged
Parts:
- Q2: renamed from Q?; footprint Package_TO_SOT_THT:TO-92_Inline -> Package_TO_SOT_THT:TO-92_Inline_Wide
- gave numbers to parts that had none: 4
Changed lines of the file:
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@@
 		(on_board yes)
 		(dnp no)
-		(property "Reference" "IN?"
+		(property "Reference" "IN2"
 			(at 74.168 72.898 90)
 			(effects
@@
 			(project "fpc"
 				(path "/01bdb219-e962-46e0-86ef-19b214cb07d2/d200b92a-1f4e-4d29-a723-683d81413cbf"
-					(reference "IN?")
+					(reference "IN2")
 					(unit 1)
 				)
@@
 		(dnp no)
 		(fields_autoplaced yes)
-		(property "Reference" "Q?"
+		(property "Reference" "Q2"
 			(at 87.63 92.7099 0)
 			(effects
@@
 			)
 		)
-		(property "Footprint" "Package_TO_SOT_THT:TO-92_Inline"
+		(property "Footprint" "Package_TO_SOT_THT:TO-92_Inline_Wide"
 			(at 87.63 95.885 0)
 			(effects
@@
 			(project "fpc"
 				(path "/01bdb219-e962-46e0-86ef-19b214cb07d2/d200b92a-1f4e-4d29-a723-683d81413cbf"
-					(reference "Q?")
+					(reference "Q2")
 					(unit 1)
 				)
@@
 		(dnp no)
 		(fields_autoplaced yes)
-		(property "Reference" "K?"
+		(property "Reference" "K2"
 			(at 111.76 72.3899 0)
 			(effects
@@
 			(project "fpc"
 				(path "/01bdb219-e962-46e0-86ef-19b214cb07d2/d200b92a-1f4e-4d29-a723-683d81413cbf"
-					(reference "K?")
+					(reference "K2")
 					(unit 1)
 				)
@@
 		(dnp no)
 		(fields_autoplaced yes)
-		(property "Reference" "R?"
+		(property "Reference" "R2"
 			(at 69.85 87.63 90)
 			(effects
@@
 			(project "fpc"
 				(path "/01bdb219-e962-46e0-86ef-19b214cb07d2/d200b92a-1f4e-4d29-a723-683d81413cbf"
-					(reference "R?")
+					(reference "R2")
 					(unit 1)
 				)
@@
 		(dnp no)
 		(fields_autoplaced yes)
-		(property "Reference" "#PWR?"
+		(property "Reference" "#PWR0101"
 			(at 85.09 59.69 0)
 			(effects
@@
 			(project "fpc"
 				(path "/01bdb219-e962-46e0-86ef-19b214cb07d2/d200b92a-1f4e-4d29-a723-683d81413cbf"
-					(reference "#PWR?")
+					(reference "#PWR0101")
 					(unit 1)
 				)
@@
 		(dnp no)
 		(fields_autoplaced yes)
-		(property "Reference" "J?"
+		(property "Reference" "J9"
 			(at 132.08 71.1199 0)
 			(effects
@@
 			(project "fpc"
 				(path "/01bdb219-e962-46e0-86ef-19b214cb07d2/d200b92a-1f4e-4d29-a723-683d81413cbf"
-					(reference "J?")
-					(unit 1)
-				)
+					(reference "J9")
+					(unit 1)
+				)
