File: marging.kicad_sch (KiCad schematic)
At the start: 23 parts, among them J4 Conn_01x04_Socket, J5 Conn_01x04_Socket, J6 Screw_Terminal_01x04, J7 Screw_Terminal_01x04, J8 15v, K1 G2RL-2, Q1 BC547, U6 DEVKIT_V1_ESP32-WROOM-32, U7 RS485_TTL_Module, U8 L7812, U9 L7805

Commit message: schematic_merged
Parts:
- removed J4, J5: Conn_01x04_Socket, symbol Connector:Conn_01x04_Socket
- removed J6, J7: Screw_Terminal_01x04, symbol Connector:Screw_Terminal_01x04
- removed U10: ~, symbol ASC712_current_sensor:ASC712_Current_sensor
- removed U7: RS485_TTL_Module, symbol rs485_ttl_sym:rs485_ttl_sm
- added D4: 1N4001, Diode_THT:D_DO-41_SOD81_P10.16mm_Horizontal, symbol Diode:1N4001
- added H1, H2, H3, H4: MountingHole_Pad, symbol Mechanical:MountingHole_Pad
- added IN2, IN3, IN4: D, symbol Device:D
- added J1, J2, J3, J4, J5: Screw_Terminal_01x04, symbol Connector:Screw_Terminal_01x04
- added J14, J15: Conn_01x04_Socket, symbol Connector:Conn_01x04_Socket
- added K2, K3, K4: G2RL-2, Relay_THT:Relay_DPDT_Omron_G2RL-2, symbol Relay:G2RL-2
- added Q2, Q3, Q4: BC547, Package_TO_SOT_THT:TO-92_Inline_Wide, symbol Transistor_BJT:BC547
- added R2, R3, R4: 1k, symbol Device:R_US
- added U1, U2, U3, U4: ~, custom:ACS712_Current_Sensor, symbol ASC712_current_sensor:ASC712_Current_sensor
- added U12: ZC261500, custom:MODULE_ZC261500, symbol ADS1115_module:ZC261500
- added U16: RS485_TTL_Module, custom:RS485_TTL, symbol rs485_ttl_sym:rs485_ttl_sm
- Q1: footprint Package_TO_SOT_THT:TO-92_Inline -> Package_TO_SOT_THT:TO-92_Inline_Wide
- U6: footprint DEVKIT_V1_ESP32-WROOM-32 (2):MODULE_DEVKIT_V1_ESP32-WROOM-32 -> custom:MODULE_DEVKIT_V1_ESP32-WROOM-32
Connections:
- net +12V: now also IN2.1 (K), IN3.1 (K), IN4.1 (K), J5.1 (Pin_1), K2.A1, K3.A1, K4.A1
- net 5V: now also U1. (GND), U2. (GND), U3. (GND), U4. (GND); no longer C15.1, C16.1, R1.1, U9.3 (OUT)
- net GND: now also H1.1, H2.1, H3.1, H4.1, J14.4 (Pin_4), J15.1 (Pin_1), J5.4 (Pin_4), Q2.3 (E), Q3.3 (E), Q4.3 (E), U1. (GND), U12.6 (ADDR), U12.9 (GND), U16. (GND), U2. (GND), U3. (GND), U4. (GND)
- net +3.3V: now reaches U6.1 (3V3)
- net +3.3V: now also J15.4 (Pin_4)
- net GPIO26: now reaches U6.10 (IO26)
- net GPIO26: now also R4.1
- net GPIO27: now reaches U6.11 (IO27)
- net GPIO27: now also R1.1
- net GPIO14: now reaches U6.12 (IO14)
- net GPIO14: now also R3.1
- net R0: now reaches U6.27 (IO16)
- net R0: now also U16. (GND)
- net D1: now reaches U6.28 (IO17)
- net D1: now also U16. (GND)
- net at U6.33 (IO21): now also U12.7 (SDA)
- net at U6.36 (IO22): now also U12.8 (SCL)
- net GPIO25: now reaches U6.9 (IO25)
- net GPIO25: now also R2.1
- net at C10.1, C9.1, D3.1 (K)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: no longer C13.1, C14.1, U9.1 (IN)
- net 15V: now reaches D3.2 (A), J8.1 (Pin_1)
- net 15V: now also D4.2 (A)
- net 3AC+: now reaches K1.11
- net 3AC+: now also J3.4 (Pin_4)
- net 3PUMP+: now reaches K1.14
- net 3PUMP+: now also J3.3 (Pin_3), U1. (GND)
- net 3AC-: now reaches K1.21
- net 3AC-: now also J3.2 (Pin_2)
- net 3pump-: now reaches K1.24
- net 3pump-: now also J3.1 (Pin_1)
- net RX: no longer names the net of U6.34 (RXD0)
- net TX: no longer names the net of U6.35 (TXD0)
- new net: IN4.2 (A), K4.A2, Q4.1 (C)
- new net: J15.2 (Pin_2), J5.3 (Pin_3)
- new net: J15.3 (Pin_3), J5.2 (Pin_2)
- new net: Q4.2 (B), R4.2
- new net: IN3.2 (A), K3.A2, Q3.1 (C)
- new net: IN2.2 (A), K2.A2, Q2.1 (C)
- new net: Q2.2 (B), R2.2
- new net: Q3.2 (B), R3.2
- new net: C13.1, C14.1, D4.1 (K), U9.1 (IN)
- new net: J14.1 (Pin_1), U16. (GND)
- new net: J14.2 (Pin_2), U16. (GND)
- new net: J14.3 (Pin_3), U16. (GND)
- new net +5V: C15.1, C16.1, U12.10 (VDD), U9.3 (OUT)
- new net 1AC+: J1.4 (Pin_4), K2.11
- new net 1AC-: J1.2 (Pin_2), K2.21
- new net 1PUMP+: J1.3 (Pin_3), K2.14, U2. (GND)
- new net 1pump-: J1.1 (Pin_1), K2.24
- new net 2AC+: J2.4 (Pin_4), K4.11
- new net 2AC-: J2.2 (Pin_2), K4.21
- new net 2PUMP+: J2.3 (Pin_3), K4.14, U4. (GND)
- new net 2pump-: J2.1 (Pin_1), K4.24
- new net 4AC+: J4.4 (Pin_4), K3.11
- new net 4AC-: J4.2 (Pin_2), K3.21
- new net 4PUMP+: J4.3 (Pin_3), K3.14, U3. (GND)
- new net 4pump-: J4.1 (Pin_1), K3.24
- new net A0: U1. (GND), U12.4 (A0)
- new net A1: U12.3 (A1), U2. (GND)
- new net A2: U12.2 (A2), U3. (GND)
- new net A3: U12.1 (A3), U4. (GND)
- no-connect marks 2 -> 38
Other:
- note removed: "Ac +"
- note removed: "Ac -"
- note removed: "Pump +"
- note removed: "Pump -"
- moved on the sheet: C10, C11, C12, C13, C14, C15, C16, C9, D3, J8, U6, U8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

Commit message: new update of schematic and pcb
Parts:
- added J13, J14, J15: Screw_Terminal_01x04, TerminalBlock_Phoenix:TerminalBlock_Phoenix_MPT-0,5-4-2.54_1x04_P2.54mm_Horizontal, symbol Connector:Screw_Terminal_01x04
- C10: renamed from C9; footprint (none) -> Capacitor_THT:CP_Radial_D5.0mm_P2.50mm
- C11: renamed from C10; footprint (none) -> Capacitor_THT:C_Disc_D4.3mm_W1.9mm_P5.00mm
- C12: renamed from C14; footprint (none) -> Capacitor_THT:C_Disc_D4.3mm_W1.9mm_P5.00mm
- C13: renamed from C11; footprint (none) -> Capacitor_THT:C_Disc_D4.3mm_W1.9mm_P5.00mm
- C14: renamed from C15; footprint (none) -> Capacitor_THT:C_Disc_D4.3mm_W1.9mm_P5.00mm
- C15: renamed from C12; footprint (none) -> Capacitor_THT:CP_Radial_D5.0mm_P2.50mm
- C16: footprint (none) -> Capacitor_THT:CP_Radial_D5.0mm_P2.50mm
- C9: renamed from C13; footprint (none) -> Capacitor_THT:CP_Radial_D5.0mm_P2.50mm
- H1, H2, H3, H4: footprint (none) -> MountingHole:MountingHole_3.2mm_M3_DIN965_Pad
- IN2: renamed from IN3; footprint (none) -> Diode_THT:D_DO-41_SOD81_P10.16mm_Horizontal
- IN3: renamed from IN1; footprint (none) -> Diode_THT:D_DO-41_SOD81_P10.16mm_Horizontal
- IN4: renamed from IN2; footprint (none) -> Diode_THT:D_DO-41_SOD81_P10.16mm_Horizontal
- IN5: renamed from IN4; footprint (none) -> Diode_THT:D_DO-41_SOD81_P10.16mm_Horizontal
- J10: renamed from J2; footprint (none) -> TerminalBlock_Phoenix:TerminalBlock_Phoenix_MPT-0,5-4-2.54_1x04_P2.54mm_Horizontal
- J11: renamed from J3; footprint (none) -> TerminalBlock_Phoenix:TerminalBlock_Phoenix_MPT-0,5-4-2.54_1x04_P2.54mm_Horizontal
- J12: renamed from J4; footprint (none) -> TerminalBlock_Phoenix:TerminalBlock_Phoenix_MPT-0,5-4-2.54_1x04_P2.54mm_Horizontal
- J5: renamed from J8; footprint (none) -> TerminalBlock:TerminalBlock_MaiXu_MX126-5.0-02P_1x02_P5.00mm
- J6: renamed from J14; footprint (none) -> Connector_PinHeader_2.54mm:PinHeader_1x04_P2.54mm_Vertical
- J7: renamed from J15; footprint (none) -> Connector_PinHeader_2.54mm:PinHeader_1x04_P2.54mm_Vertical
- J8: renamed from J5; footprint (none) -> TerminalBlock_Phoenix:TerminalBlock_Phoenix_MPT-0,5-4-2.54_1x04_P2.54mm_Horizontal
- J9: renamed from J1; footprint (none) -> TerminalBlock_Phoenix:TerminalBlock_Phoenix_MPT-0,5-4-2.54_1x04_P2.54mm_Horizontal
- R2: renamed from R3; footprint (none) -> Resistor_THT:R_Axial_DIN0207_L6.3mm_D2.5mm_P7.62mm_Horizontal
- R3: renamed from R1; footprint (none) -> Resistor_THT:R_Axial_DIN0207_L6.3mm_D2.5mm_P7.62mm_Horizontal
- R4: renamed from R2; footprint (none) -> Resistor_THT:R_Axial_DIN0207_L6.3mm_D2.5mm_P7.62mm_Horizontal
- R5: renamed from R4; footprint (none) -> Resistor_THT:R_Axial_DIN0207_L6.3mm_D2.5mm_P7.62mm_Horizontal
- U17: renamed from U16; footprint custom:RS485_TTL -> Custom:MODULE_MAX485_MODULE_5V_LOGIC_TLL_TO_RS-485_CONVERTER
- renumbered K3 to K2, K1 to K3, K2 to K4, K4 to K5, Q3 to Q2, Q1 to Q3, Q2 to Q4, Q4 to Q5, U1 to U10, U3 to U11, U8 to U12, U9 to U13, U2 to U14, U4 to U15, U6 to U16, U12 to U18
Connections:
- net +12V: now also J13.1 (Pin_1), J14.1 (Pin_1), J15.1 (Pin_1)
- net 1AC-: now also J9.3 (Pin_3); no longer J9.2 (Pin_2)
- net 1PUMP+: now also J9.1 (Pin_1), U10. (GND); no longer J9.3 (Pin_3), K4.14, U14. (GND)
- net 2AC-: now also J10.3 (Pin_3); no longer J10.2 (Pin_2)
- net 2PUMP+: now also J10.1 (Pin_1), U14. (GND); no longer J10.3 (Pin_3), K5.14, U15. (GND)
- net 3AC-: now also J11.3 (Pin_3); no longer J11.2 (Pin_2)
- net 3PUMP+: now also J11.1 (Pin_1), U11. (GND); no longer J11.3 (Pin_3), K3.14, U10. (GND)
- net 4AC-: now also J12.3 (Pin_3); no longer J12.2 (Pin_2)
- net 4PUMP+: now also J12.1 (Pin_1), U15. (GND); no longer J12.3 (Pin_3), K2.14, U11. (GND)
- net GND: now also J13.4 (Pin_4), J14.4 (Pin_4), J15.4 (Pin_4)
- net PUMP+: now reaches U15. (GND)
- net PUMP+: now also K2.14, K3.14, K4.14, K5.14, U10. (GND), U11. (GND), U14. (GND)
- net 3: now reaches J7.2 (Pin_2), J8.3 (Pin_3)
- net 3: now also J13.3 (Pin_3), J14.3 (Pin_3), J15.3 (Pin_3)
- net 2: now reaches J7.3 (Pin_3), J8.2 (Pin_2)
- net 2: now also J13.2 (Pin_2), J14.2 (Pin_2), J15.2 (Pin_2)
- net 1pump- renamed 1PUMP-
- net 1PUMP-: now also J9.2 (Pin_2); no longer J9.1 (Pin_1)
- net 2pump- renamed 2PUMP-
- net 2PUMP-: now also J10.2 (Pin_2); no longer J10.1 (Pin_1)
- net 3pump- renamed 3PUMP-
- net 3PUMP-: now also J11.2 (Pin_2); no longer J11.1 (Pin_1)
- net 4pump- renamed 4PUMP-
- net 4PUMP-: now also J12.2 (Pin_2); no longer J12.1 (Pin_1)
Other:
- moved on the sheet: J8
