File: fpc.kicad_pcb (KiCad board)
At the start: 2 copper layers, 326.1 x 122.9 mm, 75 parts, among them J1 Conn_01x15_Socket, J16 Screw_Terminal_01x04, J17 Screw_Terminal_01x04, J18 Screw_Terminal_01x04, J19 Screw_Terminal_01x04, J2 Conn_01x15_Socket, J20 Screw_Terminal_01x04, J21 Screw_Terminal_01x04, J22 15v, J3 Screw_Terminal_01x04, J4 Screw_Terminal_01x04, J5 Conn_01x02_Socket, K1 G2RL-2, K6 G2RL-2, K7 G2RL-2, K8 G2RL-2, Q1 BC547, Q6 BC547, Q7 BC547, Q8 BC547, U5 DEVKIT_V1_ESP32-WROOM-32, U6 RS485_TTL_Module, U7 ZC261500

Commit message: latest update
Parts:
- removed the ? at (266.1, 95.9)
- removed the ? at (63.7, 61.5)
- removed the ? at (313.9, 93.3)
- removed the ? at (318.1, 78.3)
- removed the ? at (60.5, 63.8)
- removed the ? at (75.6, 135.2)
- removed the ? at (264.9, 156.3)
- removed the ? at (267.9, 111.9)
- removed the ? at (267.6, 118.2)
- removed the ? at (345.6, 75.9)
- removed the ? at (345.5, 81.2)
- removed the ? at (264.7, 146.8)
- removed the ? at (114.9, 116.8)
- removed the ? at (106.5, 75.6)
- removed the ? at (67.8, 65.1)
- removed the ? at (62.8, 86.8)
- removed the ? at (348.2, 83.4)
- removed the ? at (267.2, 129.3)
- removed the ? at (335.7, 76.0)
- removed the ? at (335.7, 83.4)
- removed the ? at (264.4, 165.6)
- removed the ? at (267.2, 135.2)
- removed the ? at (314.0, 88.4)
- removed the ? at (333.1, 76.0)
- removed the ? at (134.3, 116.7)
- removed the ? at (76.5, 76.2)
- removed the ? at (333.1, 81.1)
- removed the ? at (348.2, 75.8)
- removed the ? at (83.7, 75.7)
- removed the ? at (66.3, 63.2)
- removed the ? at (318.1, 85.0)
- removed J1, J2: Conn_01x15_Socket, Connector_PinHeader_2.54mm:PinHeader_1x15_P2.54mm_Vertical
- removed K6, K7, K8: G2RL-2, Relay_THT:Relay_DPDT_Omron_G2RL-2
- added ?: , , F.Cu at (154.6, 137.2)
- added ?: , , F.Cu at (272.8, 83.0)
- added ?: , , F.Cu at (265.8, 108.0)
- added ?: , , F.Cu at (109.9, 172.8)
- added ?: , , F.Cu at (105.7, 124.2)
- added ?: , , F.Cu at (118.5, 173.5)
- added ?: , , F.Cu at (285.2, 102.0)
- added ?: , , F.Cu at (289.9, 85.4)
- added ?: , , F.Cu at (294.9, 88.7)
- added ?: , , F.Cu at (103.9, 98.7)
- added ?: , , F.Cu at (159.1, 150.5)
- added ?: , , F.Cu at (270.3, 185.6)
- added ?: , , F.Cu at (252.7, 133.2)
- added ?: , , F.Cu at (127.1, 112.3)
- added ?: , , F.Cu at (128.4, 172.3)
- added ?: , , F.Cu at (120.7, 115.8)
- added ?: , , F.Cu at (317.0, 146.5)
- added ?: , , F.Cu at (290.0, 93.5)
- added ?: , , F.Cu at (316.6, 103.1)
- added ?: , , F.Cu at (109.8, 98.8)
- added ?: , , F.Cu at (252.7, 181.7)
- added ?: , , F.Cu at (275.9, 107.1)
- added ?: , , F.Cu at (161.9, 137.2)
- added ?: , , F.Cu at (309.9, 133.9)
- added ?: , , F.Cu at (250.9, 88.9)
- added ?: , , F.Cu at (167.0, 126.9)
- added ?: , , F.Cu at (253.2, 205.3)
- added ?: , , F.Cu at (272.9, 88.7)
- added ?: , , F.Cu at (154.1, 127.2)
- added ?: , , F.Cu at (100.9, 102.1)
- added ?: , , F.Cu at (146.2, 112.5)
- added ?: , , F.Cu at (316.5, 123.6)
- added ?: , , F.Cu at (316.5, 119.7)
- added ?: , , F.Cu at (294.8, 82.8)
- added ?: , , F.Cu at (250.9, 83.1)
- added ?: , , F.Cu at (317.1, 172.9)
- added ?: , , F.Cu at (223.2, 97.1)
- added ?: , , F.Cu at (269.4, 127.7)
- added ?: , , F.Cu at (271.1, 133.6)
- added ?: , , F.Cu at (111.7, 102.0)
- added ?: , , F.Cu at (270.7, 159.2)
- added ?: , , F.Cu at (317.5, 197.9)
- added ?: , , F.Cu at (310.5, 185.5)
- added ?: , , F.Cu at (309.9, 159.4)
- added ?: , , F.Cu at (309.7, 107.6)
- added ?: , , F.Cu at (252.7, 155.3)
- added ?: , , F.Cu at (179.9, 150.4)
- added J6: Conn_01x16_Socket, Connector_PinHeader_2.54mm:PinHeader_1x16_P2.54mm_Vertical, F.Cu at (128.8, 106.3)
- added J7: Conn_01x16_Socket, Connector_PinHeader_2.54mm:PinHeader_1x16_P2.54mm_Vertical, F.Cu at (226.9, 130.9)
- added K2: Relay_SPDT, Relay_THT:Relay_SPDT_SANYOU_SRD_Series_Form_C, F.Cu at (312.0, 143.6)
- added K3: Relay_SPDT, Relay_THT:Relay_SPDT_SANYOU_SRD_Series_Form_C, F.Cu at (311.9, 169.5)
- added K4: Relay_SPDT, Relay_THT:Relay_SPDT_SANYOU_SRD_Series_Form_C, F.Cu at (312.5, 195.5)
- J16, J17, J18, J19, J20, J21, J3, J4: footprint TerminalBlock_Phoenix:TerminalBlock_Phoenix_MPT-0,5-4-2.54_1x04_P2.54mm_Horizontal -> TerminalBlock_Phoenix:TerminalBlock_Phoenix_PT-1,5-4-5.0-H_1x04_P5.00mm_Horizontal
- K1: value G2RL-2 -> Relay_SPDT; footprint Relay_THT:Relay_DPDT_Omron_G2RL-2 -> Relay_THT:Relay_SPDT_SANYOU_SRD_Series_Form_C
- U5: footprint Custom:MODULE_ESP32-DEVKITC-32E -> custom:MODULE_ESP32_NODEMCU
- moved R4 68.8 mm to (242.8, 199.2), turned to 90 degrees
- moved IN8 68.5 mm to (255.8, 200.5)
- moved IN1 67.4 mm to (255.5, 175.4)
- moved Q8 66.2 mm to (248.9, 190.3)
- moved IN7 66.0 mm to (255.6, 148.9)
- moved R2 66.0 mm to (242.6, 147.7), turned to 90 degrees
- moved R3 66.0 mm to (242.9, 173.7), turned to 90 degrees
- moved J3 65.0 mm to (260.9, 76.7)
- moved Q1 64.8 mm to (248.7, 164.9)
- moved IN6 64.7 mm to (256.0, 122.7)
- moved R1 64.1 mm to (242.6, 121.8), turned to 90 degrees
- moved Q7 63.4 mm to (248.7, 138.8)
- moved Q6 62.5 mm to (249.1, 112.7)
- moved J5 60.8 mm to (175.4, 108.0)
- moved J22 58.8 mm to (173.5, 119.5)
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Connections:
- net Net-(U6-DE) renamed /RE
- J18 pad 2: /1PUMP- -> Net-(J18-Pin_2)
- J18 pad 3: /1AC- -> Net-(J18-Pin_2)
- J19 pad 2: /2PUMP- -> Net-(J19-Pin_2)
- J19 pad 3: /2AC- -> Net-(J19-Pin_2)
- J20 pad 2: /3PUMP- -> Net-(J20-Pin_2)
- J20 pad 3: /3AC- -> Net-(J20-Pin_2)
- J21 pad 2: /4PUMP- -> Net-(J21-Pin_2)
- J21 pad 3: /4AC- -> Net-(J21-Pin_2)
- U5 pad 19: unconnected-(U5-EXT_5V-Pad19) -> +5V
- U5 pad 29: unconnected-(U5-IO5-Pad29) -> /RE+
- U5 pad 32: unconnected-(U5-GND2-Pad32) -> GND
- U5 pad 38: unconnected-(U5-GND3-Pad38) -> GND
Routing:
- net VCC: track 749.0 -> 356.9 mm
- net GND: track 531.0 -> 436.2 mm
- net /RE: track 2.54 -> 73.6 mm
- net /2: track 104.8 -> 160.0 mm
- net /R1: track 71.7 -> 19.5 mm
- net /A1: track 35.4 -> 85.3 mm
- net /A3: track 20.5 -> 64.0 mm
- net /-3PUMP+: track 56.8 -> 15.7 mm
- net /-2PUMP+: track 56.2 -> 15.7 mm
- net /-4PUMP+: track 56.6 -> 16.2 mm
- net /RE+: track 0.00 -> 40.3 mm
- net /-1PUMP+: track 55.6 -> 16.0 mm
- net /R2: track 52.8 -> 21.9 mm
- net +5V: track 161.4 -> 189.2 mm
- net /A0: track 20.2 -> 42.5 mm
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Other:
- board size 326.1 x 122.9 mm -> 251.1 x 145.4 mm
