File: fpc.kicad_pcb (KiCad board)
At the start: 2 copper layers, 268.4 x 145.4 mm, 89 parts, among them J1 Screw_Terminal_01x02, J16 Screw_Terminal_01x04, J17 Screw_Terminal_01x04, J18 Screw_Terminal_01x04, J19 Screw_Terminal_01x04, J20 Screw_Terminal_01x04, J21 Screw_Terminal_01x04, J22 15v, J3 Screw_Terminal_01x04, J4 Screw_Terminal_01x04, J5 Conn_01x02_Socket, J6 Conn_01x16_Socket, J7 Conn_01x16_Socket, K1 Relay_SPDT, K2 Relay_SPDT, K3 Relay_SPDT, K4 Relay_SPDT, Q1 BC547, Q6 BC547, Q7 BC547, Q8 BC547, U10 BUCK CONVERTER, U6 RS485_TTL_Module, U7 ZC261500, U8 ESP32-S3-DEVKIT-LIPO

Commit message: Modify schematics to one level sensor, one relay, and one current sensor.
The one current sensor may not be used for now but added in case of future
use.
Parts:
- removed ? (x44): , 
- removed H4, H5, H6, H7, H8: MountingHole_Pad, MountingHole:MountingHole_3.2mm_M3_DIN965_Pad
- removed IN1, IN6, IN8: D, Diode_THT:D_DO-41_SOD81_P10.16mm_Horizontal
- removed J16, J17, J19, J20, J21, J4: Screw_Terminal_01x04, TerminalBlock_Phoenix:TerminalBlock_Phoenix_PT-1,5-4-5.0-H_1x04_P5.00mm_Horizontal
- removed J6, J7: Conn_01x16_Socket, Connector_PinHeader_2.54mm:PinHeader_1x16_P2.54mm_Vertical
- removed K1, K3, K4: Relay_SPDT, Relay_THT:Relay_SPDT_SANYOU_SRD_Series_Form_C
- removed Q1, Q6, Q8: BC547, Package_TO_SOT_THT:TO-92_Inline
- removed R1: 220R, Resistor_THT:R_Axial_DIN0207_L6.3mm_D2.5mm_P7.62mm_Horizontal
- removed U2, U3, U4: ~, Custom:ACS712_Current_Sensor
- removed U7: ZC261500, Custom:MODULE_ZC261500
- added C1: C, Capacitor_THT:C_Disc_D5.0mm_W2.5mm_P5.00mm, F.Cu at (127.8, 96.5)
- R3, R4: value 220R -> 10K
- U1: footprint Custom:ACS712_Current_Sensor -> footprints:ACS712_Current_Sensor
- U10: footprint LM259_THT:LM2596 -> footprints:LM2596
- U6: footprint Custom:MODULE_MAX485_MODULE_5V_LOGIC_TLL_TO_RS-485_CONVERTER -> footprints:MODULE_MAX485_MODULE_5V_LOGIC_TLL_TO_RS-485_CONVERTER
- U8: footprint footprints:XCVR_ESP32-S3-DEVKIT-LIPO -> libraries:ESP32S3-DEVKIT-BOTSGEEK-LOCAL
- moved J18 258.4 mm to (98.7, 69.8), turned to 0 degrees
- moved K2 232.3 mm to (102.8, 98.2), turned to 90 degrees
- moved U1 196.7 mm to (122.0, 79.8), turned to 0 degrees
- moved IN7 186.6 mm to (92.7, 106.5), turned to 0 degrees
- moved H3 180.2 mm to (172.4, 82.3)
- moved Q7 171.5 mm to (96.8, 117.6), turned to 0 degrees
- moved R4 167.7 mm to (127.9, 102.2), turned to 180 degrees
- moved R3 164.4 mm to (121.9, 91.1), turned to 0 degrees
- moved U6 164.3 mm to (116.6, 132.3), turned to -90 degrees
- moved H2 159.0 mm to (93.3, 154.7)
- moved R2 156.8 mm to (105.6, 126.5), turned to 180 degrees
- moved J3 144.5 mm to (153.2, 155.3)
- moved J5 110.7 mm to (167.8, 69.2), turned to 90 degrees
- moved J22 102.2 mm to (182.9, 70.0), turned to 180 degrees
- moved U10 86.1 mm to (179.5, 113.6)
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Connections:
- J18 pad 1: /PUMP1_IN -> /PUMP1_OUT
- J3 pad 2: /RS485_B -> /RS485_A
- J3 pad 3: /RS485_A -> /RS485_B
- K2 pad 3: /PUMP1_OUT -> /PUMP1_IN
- R2 pad 1: /RELAY_2 -> /RELAY_1
- R3 pad 1: /RELAY_3 -> GND
- R3 pad 2: Net-(Q1-B) -> Net-(U8-GPIO5/PWR_SENS)
- R4 pad 1: /RELAY_4 -> Net-(U8-GPIO5/PWR_SENS)
- R4 pad 2: Net-(Q8-B) -> /Curr_analog_out1
- U8 pad 17: /RELAY_2 -> unconnected-(U8-GPIO17/U1TXD-Pad17)
- U8 pad 18: /RELAY_3 -> unconnected-(U8-GPIO18/U1RXD-Pad18)
- U8 pad 21: /RELAY_4 -> unconnected-(U8-GPIO21-Pad21)
- U8 pad 5: unconnected-(U8-GPIO5/PWR_SENS-PadJ1_5) -> Net-(U8-GPIO5/PWR_SENS)
- U8 pad 6: /SDA -> unconnected-(U8-GPIO6/BAT_SENS-Pad6)
- U8 pad 7: /SCL -> unconnected-(U8-GPIO7-Pad7)
- U8 pad RX: unconnected-(U8-U0RXD/GPIO44-PadJ3_3) -> (no net)
- U8 pad TX: unconnected-(U8-U0TXD/GPIO43-PadJ3_2) -> (no net)
Routing:
- net +5V: track 611.3 -> 258.4 mm
- net GND: track 259.4 -> 35.0 mm, vias 0 -> 6
- net /RELAY_4: track 164.5 -> 0.00 mm
- net /Curr_analog_out2: track 144.8 -> 0.00 mm
- net /RS485_B: track 159.8 -> 32.1 mm
- net /Curr_analog_out4: track 106.6 -> 0.00 mm
- net /RELAY_1: track 121.8 -> 35.4 mm
- net /RS485_A: track 123.1 -> 41.9 mm
- net /Curr_analog_out3: track 74.6 -> 0.00 mm
- net /DRI: track 100.2 -> 28.7 mm
- net 3.3V: track 164.6 -> 233.3 mm
- net Net-(IN6-A): track 68.2 -> 0.00 mm
- net Net-(IN1-A): track 68.0 -> 0.00 mm
- net Net-(IN8-A): track 67.6 -> 0.00 mm
- net /TX_PIN: track 94.1 -> 31.3 mm
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Other:
- board size 268.4 x 145.4 mm -> 113.1 x 106 mm

Commit message: Changes made: -Implemented a four pin terminal block to control the contactor through a Relay. -Then the pump is controlled using the contactor -Current flowing through the pump is measured using the current sensor.
NOTE: Our Relay no longer switch the pump directly, rather it switches
the contactor which in turn switches the pump.
Parts:
- removed J18: Screw_Terminal_01x04, TerminalBlock_Phoenix:TerminalBlock_Phoenix_PT-1,5-4-5.0-H_1x04_P5.00mm_Horizontal
- added Contactor1: Screw_Terminal_01x04, TerminalBlock_Phoenix:TerminalBlock_Phoenix_PT-1,5-4-5.0-H_1x04_P5.00mm_Horizontal, F.Cu at (95.5, 70.0)
Connections:
- K2 pad 1: /Power_Source_1 -> /Contactor_live_in
- K2 pad 3: /PUMP1_IN -> /Contactor_live_out
- U1 pad 5: /PUMP1_OUT -> /Pump_live_out
- U1 pad 6: /PUMP1_IN -> /Pump_live_in
Routing:
- net /Power_Source_1: track 67.0 -> 0.00 mm
- net /Contactor_live_in: track 0.00 -> 52.0 mm
- net /PUMP1_OUT: track 35.1 -> 0.00 mm
- net /Pump_live_in: track 0.00 -> 23.4 mm
- net /Contactor_live_out: track 0.00 -> 23.1 mm
- net /PUMP1_IN: track 19.8 -> 0.00 mm
- net /Pump_live_out: track 0.00 -> 14.6 mm
- net /Neutral_1: track 5.00 -> 0.00 mm
