File: fpc.kicad_sch (KiCad schematic)
At the start: 45 parts, among them J16 Screw_Terminal_01x04, J17 Screw_Terminal_01x04, J18 Screw_Terminal_01x04, J19 Screw_Terminal_01x04, J20 Screw_Terminal_01x04, J21 Screw_Terminal_01x04, J22 15v, J3 Screw_Terminal_01x04, J4 Screw_Terminal_01x04, J5 Conn_01x02_Socket, J6 Conn_01x16_Socket, J7 Conn_01x16_Socket, K1 Relay_SPDT, K2 Relay_SPDT, K3 Relay_SPDT, K4 Relay_SPDT, Q1 BC547, Q6 BC547, Q7 BC547, Q8 BC547, SW1 SW_Push, U5 DEVKIT_V1_ESP32-WROOM-32, U6 RS485_TTL_Module, U7 ZC261500

Commit message: - Changing of PCB Layout - Change the microcontroller from ESP32 to ESP32 S3 - Reroute the board
Parts:
- removed SW1: SW_Push, symbol Switch:SW_Push
- removed U5: DEVKIT_V1_ESP32-WROOM-32, custom:MODULE_ESP32_NODEMCU, symbol DEVKIT_V1_ESP32-WROOM-32:DEVKIT_V1_ESP32-WROOM-32
- added U5: ESP32-S3-DEVKITC-1U-N8R8, RF_Module:MODULE_ESP32-S3-DEVKITC-1U-N8R8, symbol MCU_Espressif:ESP32-S3-DEVKITC-1U-N8R8
- U1, U10, U2, U3, U4: value ~ -> (none)
Connections:
- net D1+ is gone; now on net RX_PIN: J6.10 (Pin_10)
- net GPIO25 is gone; now on net GPIO14: J6.1 (Pin_1)
- net R0+ is gone; now on net DRI: J6.11 (Pin_11)
- net +5V: now also U5.J1_21 (5V0)
- net 3.3V: now also U5.J1_1 (3V3), U5.J1_2 (3V3__1)
- net GND: now also U5.J1_22 (GND), U5.J3_1 (GND__1), U5.J3_21 (GND__2), U5.J3_22 (GND__3)
- net GPIO14: now also U5.J1_20 (GPIO14); no longer J6.7 (Pin_7)
- net GPIO4: now also U5.J1_4 (GPIO4)
- net SDA: now reaches U7.7 (SDA)
- net SDA: now also U5.J1_6 (GPIO6)
- net SCL: now reaches U7.8 (SCL)
- net SCL: now also U5.J1_7 (GPIO7)
- net D1 renamed RX_PIN
- net RX_PIN: now also U6.1 (R0), U5.J1_17 (GPIO11); no longer U6.4 (DI)
- net GPIO26 renamed GPIO17
- net GPIO17: now also U5.J1_10 (GPIO17)
- net GPIO27 renamed GPIO18
- net GPIO18: now also U5.J1_11 (GPIO18)
- net R0 renamed DRI
- net DRI: now also U6.2 (RE), U6.3 (DE), U5.J1_15 (GPIO9); no longer U6.1 (R0)
- net R1 renamed RELAY_1
- net R2 renamed RELAY_2
- net R3 renamed RELAY_3
- net R4 renamed RELAY_4
- removed net RE: J7.12 (Pin_12), U6.2 (RE), U6.3 (DE)
- net RE+ renamed TX_PIN
- net TX_PIN: now also J7.12 (Pin_12), U6.4 (DI), U5.J1_16 (GPIO10)
- new net GPIO21: J6.7 (Pin_7), U5.J3_18 (GPIO21)
- no-connect marks 34 -> 37
Other:
- moved on the sheet: J6, U6
