File: fpc.kicad_sch (KiCad schematic)
At the start: 19 parts, among them J1 Screw_Terminal_01x02, J18 Screw_Terminal_01x04, J22 15v, J3 Screw_Terminal_01x04, J5 Conn_01x02_Socket, K2 Relay_SPDT, Q7 BC547, U10 BUCK CONVERTER, U6 RS485_TTL_Module, U8 ESP32-S3-DEVKIT-LIPO

Commit message: Changes made: -Implemented a four pin terminal block to control the contactor through a Relay. -Then the pump is controlled using the contactor -Current flowing through the pump is measured using the current sensor.
NOTE: Our Relay no longer switch the pump directly, rather it switches
the contactor which in turn switches the pump.
Parts:
- removed J18: Screw_Terminal_01x04, TerminalBlock_Phoenix:TerminalBlock_Phoenix_PT-1,5-4-5.0-H_1x04_P5.00mm_Horizontal, symbol Connector:Screw_Terminal_01x04
- added Contactor1: Screw_Terminal_01x04, TerminalBlock_Phoenix:TerminalBlock_Phoenix_PT-1,5-4-5.0-H_1x04_P5.00mm_Horizontal, symbol Connector:Screw_Terminal_01x04
Connections:
- net +3V3: no longer U8.J1_2 (+3V3)
- net GND: no longer U8.J3_1 (GND), U8.J3_21 (GND), U8.J3_22 (GND)
- net PUMP1_IN renamed Contactor_live_out
- net Contactor_live_out: now also Contactor1.1 (Pin_1); no longer U1.6 (IP+(I_in))
- net PUMP1_OUT renamed Pump_live_out
- net Pump_live_out: now also Contactor1.4 (Pin_4)
- net Power_Source_1 renamed Contactor_live_in
- net Contactor_live_in: now also Contactor1.2 (Pin_2)
- new net Pump_live_in: Contactor1.3 (Pin_3), U1.6 (IP+(I_in))

Commit message: A buzzer circuit was included in the circuit to notify users in case of faulty sensor, no change in rise level e.t.c
Parts:
- added J2: BUZZER, Connector_JST:JST_EH_B2B-EH-A_1x02_P2.50mm_Vertical, symbol Connector:Conn_01x02_Pin
- added Q1: BC547, Library:BC547-BOTSGEEK, symbol Transistor_BJT:BC547
- added R1: 220R, Resistor_THT:R_Axial_DIN0207_L6.3mm_D2.5mm_P7.62mm_Horizontal, symbol Device:R_US
- Q7: footprint Package_TO_SOT_THT:TO-92_Inline -> Library:BC547-BOTSGEEK
Connections:
- net +5V: now also J2.1 (Pin_1)
- net GND: now also Q1.3 (E)
- net BUZZER_PIN: now reaches U8.7 (GPIO7)
- net BUZZER_PIN: now also R1.1
- new net: Q1.2 (B), R1.2
- new net BUZZER_NEG_PIN: J2.2 (Pin_2), Q1.1 (C)
- no-connect marks 33 -> 32
Other:
- note added: "BUZZER CIRCUIT"
